File: rp2350.kicad_sch (KiCad schematic)
At the start: 32 parts, among them J20 Conn_01x03, U5 RP2350-QFN80, U6 W25Q32JVSS, Y1 12.0MHz

Commit message: v3.2 as prototyped
Parts:
- C26: renamed from C44; JLC (none) -> C325455
- C27: renamed from C48; Characteristics (none) -> 100n 10% 25V XR 0402; JLC (none) -> C100072; LCSC (none) -> C100072; MPN (none) -> CL05A104KA5NNNC
- C28: renamed from C45; JLC (none) -> C325455
- C29: renamed from C31; Characteristics (none) -> 100n 10% 25V XR 0402; JLC (none) -> C100072; LCSC (none) -> C100072; MPN (none) -> CL05A104KA5NNNC
- C30: renamed from C32; Characteristics (none) -> 4.7u 0402; JLC (none) -> C2858031; MPN (none) -> GRM155R61E475ME15D
- C31: renamed from C33; Characteristics (none) -> 100n 10% 25V XR 0402; JLC (none) -> C100072; LCSC (none) -> C100072; MPN (none) -> CL05A104KA5NNNC
- C32: renamed from C38; Characteristics (none) -> 100n 10% 25V XR 0402; JLC (none) -> C100072; LCSC (none) -> C100072; MPN (none) -> CL05A104KA5NNNC
- C33: renamed from C40; Characteristics (none) -> 100n 10% 25V XR 0402; JLC (none) -> C100072; LCSC (none) -> C100072; MPN (none) -> CL05A104KA5NNNC
- C34: renamed from C42; Characteristics (none) -> 100n 10% 25V XR 0402; JLC (none) -> C100072; LCSC (none) -> C100072; MPN (none) -> CL05A104KA5NNNC
- C35: renamed from C46; Characteristics (none) -> 100n 10% 25V XR 0402; JLC (none) -> C100072; LCSC (none) -> C100072; MPN (none) -> CL05A104KA5NNNC
- C36: renamed from C47; Characteristics (none) -> 100n 10% 25V XR 0402; JLC (none) -> C100072; LCSC (none) -> C100072; MPN (none) -> CL05A104KA5NNNC
- C37: Characteristics (none) -> 100n 10% 25V XR 0402; JLC (none) -> C100072; LCSC (none) -> C100072; MPN (none) -> CL05A104KA5NNNC
- C38: renamed from C39; Characteristics (none) -> 100n 10% 25V XR 0402; JLC (none) -> C100072; LCSC (none) -> C100072; MPN (none) -> CL05A104KA5NNNC
- C39: renamed from C41; Characteristics (none) -> 100n 10% 25V XR 0402; JLC (none) -> C100072; LCSC (none) -> C100072; MPN (none) -> CL05A104KA5NNNC
- C40: renamed from C43; Characteristics (none) -> 100n 10% 25V XR 0402; JLC (none) -> C100072; LCSC (none) -> C100072; MPN (none) -> CL05A104KA5NNNC
- C41: renamed from C36; Characteristics (none) -> 4.7u 0402; JLC (none) -> C2858031; MPN (none) -> GRM155R61E475ME15D
- C42: renamed from C34; Characteristics (none) -> 4.7u 0603; JLC (none) -> C237615; MPN (none) -> GRM188C71C475KE21D
- C43: renamed from C35; Characteristics (none) -> 4.7u 0603; JLC (none) -> C237615; MPN (none) -> GRM188C71C475KE21D
- L1: Characteristics (none) -> 0806 Power Inductors; JLC (none) -> C42411119
- R54: renamed from R44; Characteristics (none) -> 27R 0402; JLC (none) -> C2098172; MPN (none) -> AF0402FR-0727RL
- R55: renamed from R45; Characteristics (none) -> 27R 0402; JLC (none) -> C2098172; MPN (none) -> AF0402FR-0727RL
- R56: renamed from R49; JLC (none) -> C25744
- R57: renamed from R47; JLC (none) -> C11702
- R58: renamed from R48; JLC (none) -> C17168
- R59: renamed from R46; value 33 -> 33R; Characteristics (none) -> 33R 0402; JLC (none) -> C25105; MPN (none) -> RCS040233R0FKED
- U3: renamed from U5; Characteristics (none) -> QFN-80-EP(10x10) Microcontroller; JLC (none) -> C42415655; MPN (none) -> RP2350B
- U4: renamed from U6; Characteristics (none) -> W25Q32 Flash; JLC (none) -> C82344; MPN (none) -> W25Q32JVSSIQ
- Y1: JLC (none) -> C255902
- renumbered J20 to J15, LAYOUT2 to LAYOUT1, LAYOUT3 to LAYOUT2, LAYOUT1 to LAYOUT3
Connections:
- net ADC0 renamed GPIO40
