File: tinytapeout-demo.kicad_sch (KiCad schematic)
At the start: 127 parts, among them J1 Conn_01x06, J12 613012243121, J13 613012243121, J14 613012243121, J16 2x20_P2.54mm_Pinheader, J17 Conn_01x03, J18 2x20_P2.54mm_Pinheader, J19 Conn_01x02, J2 Conn_01x04, J20 USB_C, J3 613012243121, J4 TT06_BREAKOUT_REVA, J5 613012243121, J6 613012243121, J7 Conn_01x02, J8 Conn_01x03, J9 Conn_01x16, Q1 DMN2005K, SW1 434121025816, SW2 434121025816, SW3 434121025816, SW4 193-8MSR, U1 157112V12700, U2 TLV1117LV33, U3 AP2112K-1.8

Commit message: nextgen v3 PRELIMINARY
Parts:
- removed C11, C5, C57, C59, C61: 1uF, Capacitor_SMD:C_0603_1608Metric, symbol Device:C_Small
- removed C13, C4, C56, C58, C60, C8: 100nF, Capacitor_SMD:C_0402_1005Metric, symbol Device:C_Small
- removed C45, C46, C47: C_33p_0402_50V, Capacitor_SMD:C_0402_1005Metric, symbol psypassives:C_33p_0402_50V
- removed C6, C7: 10uF, Capacitor_SMD:C_0805_2012Metric, symbol Device:C_Small
- removed D3: Yellow, LED_SMD:LED_0603_1608Metric, symbol Device:LED_Small
- removed J1: Conn_01x06, Connector_PinHeader_2.54mm:PinHeader_1x06_P2.54mm_Vertical, symbol Connector_Generic:Conn_01x06
- removed J12, J13, J14, J3: 613012243121, TinyTapeout:PinSocket_2x06_P2.54mm_PMODHost1A, symbol TinyTapeout:PMOD_HOST_2x6
- removed J19: Conn_01x02, Connector_PinHeader_2.54mm:PinHeader_1x02_P2.54mm_Vertical, symbol Connector_Generic:Conn_01x02
- removed J2: Conn_01x04, Connector_PinHeader_2.54mm:PinHeader_1x04_P2.54mm_Vertical, symbol Connector_Generic:Conn_01x04
- removed J4: TT06_BREAKOUT_REVA, TinyTapeout:TT06_CARRIER_ON_DB, symbol TinyTapeout:OPENFRAME_TT06_BREAKOUT_REVA
- removed J7: Conn_01x02, Connector_PinHeader_2.54mm:PinHeader_1x02_P2.54mm_Vertical_SMD_Pin1Right, symbol Connector_Generic:Conn_01x02
- removed J8: Conn_01x03, Connector_PinHeader_2.54mm:PinHeader_1x03_P2.54mm_Vertical, symbol Connector_Generic:Conn_01x03
- removed Q1: DMN2005K, Package_TO_SOT_SMD:SOT-23, symbol psychogenic:DMN2005K
- removed R12: 10k, Resistor_SMD:R_0402_1005Metric, symbol Device:R_Small
- removed R20: 5.1k, Resistor_SMD:R_0402_1005Metric, symbol Device:R_Small
- removed R22, R23, R24, R25, R26, R27: 510, Resistor_SMD:R_0402_1005Metric, symbol Device:R_Small
- removed R3, R4, R5, R6: 1k, Resistor_SMD:R_0402_1005Metric, symbol Device:R_Small
- removed R42, R44, R45, R46, R47, R48, R51, R52, R53, R54, R55: 1M, Resistor_SMD:R_0402_1005Metric, symbol Device:R_Small
- removed R49: 0R, Resistor_SMD:R_0603_1608Metric, symbol Device:R_Small
- removed R50: 47R, Resistor_SMD:R_0402_1005Metric, symbol Device:R_Small
- removed R7: 47k, Resistor_SMD:R_0603_1608Metric, symbol Device:R_Small
- removed U1: 157112V12700, TinyTapeout:WL_S7DS-157112V12700, symbol Display_Character:KCSC02-106
- removed U2: TLV1117LV33, Package_TO_SOT_SMD:SOT-223-3_TabPin2, symbol Regulator_Linear:AZ1117-3.3
- removed U3: AP2112K-1.8, Package_TO_SOT_SMD:SOT-23-5, symbol Regulator_Linear:AP2112K-1.8
- added C10: 1uF, Capacitor_SMD:C_0603_1608Metric, symbol Device:C_Small
- added C12: 10uF, Capacitor_SMD:C_0805_2012Metric, symbol Device:C_Small
- added C17, C9: 100nF, Capacitor_SMD:C_0402_1005Metric, symbol Device:C_Small
- added C4, C6, C8: C_33p_0402_50V, Capacitor_SMD:C_0402_1005Metric, symbol psypassives:C_33p_0402_50V
- added J1: TT_HRS_BREAKOUT_REVA, TinyTapeout:TT_HRS_CARRIER_REVA, symbol TinyTapeout:TT_HRS_BREAKOUT_REVA
- added J11, J12, J3, J4: DF40C-20DS-0.4V_51, TinyTapeout:HRS_DF40C-20DP-0.4V_51, symbol TinyTapeout:DF40C-20DP-0.4V_51
- added J13: Conn_01x03, Connector_PinHeader_2.54mm:PinHeader_1x03_P2.54mm_Vertical, symbol Connector_Generic:Conn_01x03
- added J15, J16: Conn_01x04, Connector_PinHeader_2.54mm:PinHeader_1x04_P2.54mm_Vertical, symbol Connector_Generic:Conn_01x04
- added J2: Conn_01x02, Connector_PinHeader_2.54mm:PinHeader_1x02_P2.54mm_Vertical, symbol Connector_Generic:Conn_01x02
- added J6: 613012243121, TinyTapeout:PinSocket_2x06_P2.54mm_PMODHost1A, symbol TinyTapeout:PMOD_HOST_2x6
- added LAYOUT4: Standardized layout to allow for dual expansion b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, symbol psychogenic:LAYOUT
- added R12, R13, R19, R20, R23, R24, R25, R26, R4, R5, R6, R7: 1M, Resistor_SMD:R_0402_1005Metric, symbol psycomponents:PsyResistors_IEC/R_1M_0402_1005-14
- added R14: 1k, Resistor_SMD:R_0402_1005Metric, symbol Device:R_Small
- added R28: 1M, Resistor_SMD:R_0603_1608Metric, symbol Device:R_Small
- added R29, R30: 5.1k, Resistor_SMD:R_0402_1005Metric, symbol Device:R_Small
- added R32, R33, R34, R35, R36, R37: 510, Resistor_SMD:R_0402_1005Metric, symbol Device:R_Small
- added R41: 1.2K, Resistor_SMD:R_0402_1005Metric, symbol Device:R_Small
- added U1: TLV1117LV33, Package_TO_SOT_SMD:SOT-223-3_TabPin2, symbol Regulator_Linear:AZ1117-3.3
- added U2: 157112V12700, TinyTapeout:WL_S7DS-157112V12700, symbol Display_Character:KCSC02-106
- JP1, JP2, JP3, JP4, JP5, JP6, JP7, JP8: footprint TinyTapeout:SolderJumper-2_Bridged_Throughole1 -> TinyTapeout:SolderJumper-2_0603
- R10: value 1k -> 47k; Characteristics 1k 0402 -> 47k 0402; LCSC C202394 -> (none); MPN CR0402-FX-1001GLF -> (none); MPN_ALT WR04X1001FTL -> (none)
- R15: value 1.2K -> 1k; Characteristics 1.2k 0402 -> 1k 0402; LCSC C138040 -> C202394; MPN RC0402FR-071K2L -> CR0402-FX-1001GLF; MPN_ALT CR0402-JW-122GLF -> WR04X1001FTL
- R16: value 1M -> 1k; footprint Resistor_SMD:R_0603_1608Metric -> Resistor_SMD:R_0402_1005Metric; Characteristics 1M 0603 -> 1k 0402; LCSC C858907 -> C202394; MPN (none) -> CR0402-FX-1001GLF; MPN_ALT (none) -> WR04X1001FTL; now fitted
- R17, R18: value 510 -> 10k; Characteristics 510R 0402 -> 10k 0402; LCSC C276273 -> C471764; MPN RC0402FR-07510RL -> RC0402FR-0710KL; MPN_ALT CR0402-FX-5100GLF -> WR04X1002FTL
- R2: value 1k -> 10k; Characteristics 1k 0402 -> 10k 0402; LCSC C202394 -> C471764; MPN CR0402-FX-1001GLF -> RC0402FR-0710KL; MPN_ALT WR04X1001FTL -> WR04X1002FTL
- R21: value 5.1k -> 1k; Characteristics 5.1k 0402 -> 1k 0402; LCSC C138073 -> C202394; MPN AC0402FR-135K1L -> CR0402-FX-1001GLF; MPN_ALT CR0402-FX-5101GLF -> WR04X1001FTL
- R43: value 1M -> 510; Characteristics 1M 0402 -> 510R 0402; LCSC C138033 -> C276273; MPN CR0402-FX-1004GLF -> RC0402FR-07510RL; MPN_ALT RC0402FR-071ML -> CR0402-FX-5100GLF
- R8, R9: value 10k -> 1k; Characteristics 10k 0402 -> 1k 0402; LCSC C471764 -> C202394; MPN RC0402FR-0710KL -> CR0402-FX-1001GLF; MPN_ALT WR04X1002FTL -> WR04X1001FTL
- renumbered C49 to C11, C16 to C13, C17 to C14, C21 to C15, C25 to C16, C26 to C18, C10 to C19, C9 to C20, C12 to C21, C24 to C22, C14 to C24, C15 to C25, C44 to C5, C48 to C7, D5 to D1, D6 to D2, D1 to D3, D2 to D4, J6 to J10, J17 to J14, J9 to J17, J20 to J5, J16 to J7, J18 to J8, J5 to J9, R13 to R22, R41 to R27, R14 to R3, R30 to R31, R28 to R38, R29 to R39, R31 to R40, R32 to R42, SW3 to SW1, SW1 to SW2, SW2 to SW3
Connections:
- net RPIO29 is gone; now on net +3V3: J17.14 (Pin_14)
- net an4 is gone; now on net +3V3: R43.1
- net +3V3: now also C22.2, R15.1, R16.1, R21.1, C10.2, C17.1, C9.1, J1.L8 (3v3), J1.R5 (3v3), J11.3, J12.3, J3.3, J4.3, J6.12 (VCC), J6.6 (VCC), R14.1, U1.2 (VO); no longer C18.2, R10.1, R17.1
- net CC1: now also C6.1, R30.1; no longer R21.1
- net CC2: now also C4.1, R29.1
- net GND: now also R10.2, C10.1, C12.2, C17.2, C4.2, C6.2, C8.2, C9.2, J1.L11 (GND), J1.L16 (GND), J1.L17 (GND), J1.L2 (GND), J1.L22 (GND), J1.L24 (GND), J1.L26 (GND), J1.L28 (GND), J1.L30 (GND), J1.L31 (GND), J1.L32 (GND), J1.L34 (GND), J1.L37 (GND), J1.L38 (GND), J1.L6 (GND), J1.R11 (GND), J1.R14 (GND), J1.R15 (GND), J1.R17 (GND), J1.R19 (GND), J1.R2 (GND), J1.R21 (GND), J1.R23 (GND), J1.R25 (GND), J1.R27 (GND), J1.R28 (GND), J1.R33 (GND), J1.R34 (GND), J1.R39 (GND), J1.R4 (GND), J1.R40 (GND), J1.R45 (GND), J1.R46 (GND), J1.R49 (GND), J1.R50 (GND), J1.R6 (GND), J1.R8 (GND), J11.12, J11.13, J11.2, J11.20, J11.8, J12.12, J12.13, J12.2, J12.20, J12.8, J2.1 (Pin_1), J3.10, J3.12, J3.13, J3.14, J3.16, J3.18, J3.2, J3.20, J3.4, J3.5, J3.6, J3.8, J4.10, J4.12, J4.13, J4.14, J4.16, J4.18, J4.2, J4.20, J4.4, J4.5, J4.6, J4.8, J6.11 (GND), J6.5 (GND), R12.1, R13.1, R19.1, R20.1, R23.2, R24.2, R25.2, R26.2, R28.2, R29.2, R30.2, R4.2, R5.2, R6.2, R7.2, U1.1 (GND), U2.3 (CC), U2.8 (CC); no longer R16.2, R21.2, R43.2
- net VBUS: now also C11.1, C15.2, C16.2, C18.2, FB1.2, J17.16 (Pin_16), C12.1, J1.R1 (VBUS), J1.R3 (VBUS), J11.1, J12.1, J3.1, J4.1, R41.1, U1.3 (VI); no longer F1.1, J5.A4 (VBUS), J5.A9 (VBUS), J5.B4 (VBUS), J5.B9 (VBUS)
- net ctrl_ena: now also J17.8 (Pin_8), J1.L1 (ctrl_ena); no longer J17.6 (Pin_6)
- net ctrl_sel_inc: now also J17.7 (Pin_7), J1.L4 (ctrl_inc); no longer J17.8 (Pin_8)
- net project_clk: now also R17.1, J1.L36 (proj_clk)
- net res1: now also J17.12 (Pin_12), J1.L5 (RES1); no longer J17.10 (Pin_10)
- net res2: now also J1.L7 (RES2)
- net res3: now also J17.10 (Pin_10), J1.L9 (RES3); no longer J17.12 (Pin_12)
- net ui_in0: now also J1.L10 (ui_in[0]), J15.1 (Pin_1), J6.1 (IO1)
- net ui_in1: now also J1.L12 (ui_in[1]), J15.2 (Pin_2), J6.2 (IO2)
- net ui_in2: now also J1.L13 (ui_in[2]), J15.3 (Pin_3), J6.3 (IO3)
- net ui_in3: now also J1.L14 (ui_in[3]), J15.4 (Pin_4), J6.4 (IO4)
- net ui_in4: now also J1.L18 (ui_in[4]), J6.7 (IO5)
- net ui_in5: now also J1.L20 (ui_in[5]), J6.8 (IO6)
- net ui_in6: now also J1.L15 (ui_in[6]), J6.9 (IO7)
- net ui_in7: now also J1.L33 (ui_in[7]), J6.10 (IO8)
- net uio0: now also J1.L40 (uio[0]), J13.1 (Pin_1)
- net uio1: now also J1.L39 (uio[1]), J13.2 (Pin_2)
- net uio2: now also J1.R48 (uio[2]), J13.3 (Pin_3)
- net uio3: now also J1.R47 (uio[3])
- net uio4: now also J1.R44 (uio[4])
- net uio5: now also J1.R43 (uio[5])
- net uio6: now also J1.R42 (uio[6])
- net uio7: now also J1.R41 (uio[7])
- net uo_out0: now also J1.R38 (uo_out[0]), J16.1 (Pin_1)
- net uo_out1: now also J1.R37 (uo_out[1]), J16.2 (Pin_2)
- net uo_out2: now also J1.R36 (uo_out[2]), J16.3 (Pin_3)
- net uo_out3: now also J1.R35 (uo_out[3]), J16.4 (Pin_4)
- net uo_out4: now also J1.R32 (uo_out[4])
- net uo_out5: now also J1.R31 (uo_out[5])
- net uo_out6: now also J1.R30 (uo_out[6])
- net uo_out7: now also J1.R29 (uo_out[7])
- net usb_d+: now also C8.1
- net ~{ctrl_sel_rst}: now also J17.6 (Pin_6), J1.L3 (ctrl_~{rst}); no longer J17.7 (Pin_7)
- net ~{project_rst}: now also J1.L35 (proj_~{rst})
- net at C1.2, SW2.1: now also R10.1, R17.2
- net at R22.1, SW3.2: now also R18.2; no longer R8.2
- net at JP5.2 (B): now also R36.1
- net at JP2.2 (B): now also R33.1
- net at SW4.4: now also R14.2
- net at D4.2 (A): now also R43.2; no longer R17.2
- net at SW4.3: now also R15.2
- net at SW4.1: now also R21.2; no longer R11.2
- net at SW4.2: now also R16.2; no longer R10.2
- net at SW4.5: now also R11.2
- net at SW4.6: now also R9.2
- net at SW4.7: now also R8.2; no longer R2.2
- net at R38.2: now also U2.10 (G)
- net at R39.2: now also U2.5 (DP)
- net at JP4.2 (B): now also R35.1
- net at JP1.2 (B): now also R32.1
- net at JP6.2 (B): now also R37.1
- net at JP3.2 (B): now also R34.1
- net at D3.2 (A): now also R41.2; no longer R15.2
- net at C3.1, J5.S1 (SHIELD): now also R28.1; no longer R16.1
- removed net +1V8: C15.2, C16.2, C22.2, J17.4 (Pin_4)
- removed net +5V: C11.1, FB1.2, J17.16 (Pin_16), R15.1
- net boot_mode renamed BOOT
- net BOOT: now also R2.2; no longer R9.2
- new net: R35.2, U2.2 (D)
- new net: R36.2, U2.1 (E)
- new net: R34.2, U2.4 (C)
- new net: R33.2, U2.6 (B)
- new net: R32.2, U2.7 (A)
- new net: R37.2, U2.9 (F)
- new net ADC0: J11.15, J12.15
- new net ADC1: J11.17, J12.17
- new net ADC2: J11.19, J12.19
- new net ADC3: J11.18, J12.18
- new net ADC4: J11.16, J12.16
- new net ADC5: J11.14, J12.14
- new net CS: J11.7, J12.7
- new net IO29: J11.9, J12.9
- new net IO30: J11.10, J12.10
- new net IO31: J11.11, J12.11
- new net MISO: J11.4, J12.4
- new net MOSI: J11.5, J12.5
- new net RUN: J2.2 (Pin_2)
- new net SCK: J11.6, J12.6
- new net VBUSRW: F1.1, J5.A4 (VBUS), J5.A9 (VBUS), J5.B4 (VBUS), J5.B9 (VBUS)
- new net analog0: J1.L19 (an0), J4.7, R12.2
- new net analog1: J1.L21 (an1), J4.9, R13.2
- new net analog10: J1.R18 (an10), J3.17, R25.1
- new net analog11: J1.R16 (an11), J3.19, R26.1
- new net analog2: J1.L23 (an2), J4.11, R4.1
- new net analog3: J1.L25 (an3), J4.15, R5.1
- new net analog4: J1.L27 (an4), J4.17, R6.1
- new net analog5: J1.L29 (an5), J4.19, R7.1
- new net analog6: J1.R26 (an6), J3.7, R19.2
- new net analog7: J1.R24 (an7), J3.9, R20.2
- new net analog8: J1.R22 (an8), J3.11, R23.1
- new net analog9: J1.R20 (an9), J3.15, R24.1
- new net m_ADC: J1.R7 (ADC)
- new net m_CS: J1.R12 (CS)
- new net m_RX: J1.R13 (RX)
- new net m_SCK: J1.R9 (SCK)
- new net m_TX: J1.R10 (TX)
Other:
- removed sheet RP2040
- added sheet RP2350 (rp2350.kicad_sch)
- note added: "ASIC I/O"
- note added: "All analog pins pulled down on DB"
- note added: "Analog Bank A"
- note added: "Analog Bank B"
- note added: "Expansion headers placed on each side, in line with analog, 10mm to right when facing breakout."
- note added: "Project Control"
- note added: "RP2350B"
- note added: "Short to hold RP2 in reset"
- note added: "Tiny Tapeout Demoboard v3 (PRELIMINARY)"
- note removed: "1.8V LDO"
- note removed: "50mA hold fuse removed"
- note removed: "Analog pins are held low to ensure nice state. Jumpers on carrier may be cut to get rid of the header traversal and termination."
- note removed: "CS"
- note removed: "Changed to smaller SOT-23 LDO for core supply. If using the 2112, can still get up to 600mA which is more than we need and should be safe for external draw."
- note removed: "Control"
- note removed: "Core power profiling possible by either removing R49 and metering current through J19 pads or replacing R49 with non-zero value and measuring V across using J19, coulomb counter style."
- note removed: "DI"
- note removed: "DO"
- note removed: "E.g. if you wanted an SPI controlled periph as part of your TT project, you could configure it such that it uses: in[0] as select/~{cs} in[1] for clocking in[2] for tx/copi and out[3] for rx/cipo"
- note removed: "For reference, digilent standard pinouts"
- note removed: "I/O"
- note removed: "I2C"
- note removed: "I2C1"
- note removed: "PMOD Standard Pinouts"
- note removed: "PMOD, specialized versions. These PMODs offer an array of options while attempting to keep to standard digilent pinouts. With "SPI Periph", the pmod controls the bus and the project responds. On "SPI Control", the pmod is a peripheral device to the project. The bidir/uart header is flexible."
- note removed: "Pinout follows non-numerical ordering in order to support various standard communications methods between IC and projects. In yellow, possible mappings for SPI, I2C and UART, from RP2040 perspective. See in sheet for full mapping."
- note removed: "Place C close to relevant supply"
- note removed: "Possible Comms"
- note removed: "RP2040 MCU"
- note removed: "RX"
- note removed: "SCK"
- note removed: "SPI"
- note removed: "SPI Bi/UART"
- note removed: "SPI Control/I2C"
- note removed: "SPI Periph"
- note removed: "SPI-Bi"
- note removed: "SPI-MA"
- note removed: "SPI-MB"
- note removed: "SPI-SA"
- note removed: "SPI-SB"
- note removed: "SPI0"
- note removed: "SPI1"
- note removed: "SPI1 UART1 I2C0 I2C1"
- note removed: "TT Carrier Logic"
- note removed: "TT Carrier Power"
- note removed: "TT06+ Demoboard: TT06+ breakout pinout, piano dip, indicators for levering out the breakout, TT-standard naming of ports."
- note removed: "TX"
- note removed: "Tiny Tapeout 06+ Demo Board"
- note removed: "UART"
- note removed: "UART0"
- note removed: "USER-FACING CHANGES from TT04 * top header (J9) shorter, pin changes * no demoboard MUX in the way of low out nibble * more comfortable input DIP (rocker or piano, TBD) All RP2040 pin mappings for I/O are the same. All PMOD connectors are the same. Project reset and ASIC MUX pins have moved, but will be transparent for SDK users. MAJOR Changes from TT04 * carrier board new size and pinout * analo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"
- note removed: "ci"
- note removed: "cipo"
- note removed: "co"
- note removed: "copi"
- note removed: "cs"
- note removed: "cs(m)"
- note removed: "cts"
- note removed: "i2c eeprom on carrier 2: SDA1 3: SCL1"
- note removed: "mi"
- note removed: "mi(m)"
- note removed: "mo"
- note removed: "mo(m)"
- note removed: "rts"
- note removed: "rx"
- note removed: "sck"
- note removed: "sck(m)"
- note removed: "tx"
- note removed: "urx"
- note removed: "utx"
- company: Psychogenic Technologies -> Psychogenic Technologies INC
- title: Tiny Tapeout 06+ Demo Board -> Tiny Tapeout Demoboard v3 (PRELIMINARY)
- moved on the sheet: C1, C11, C13, C14, C15, C16, C18, C19, C2, C20, C21, C22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

Commit message: v3.2 as prototyped
Parts:
- removed unit 5 of J1
- removed J11, J12, J3, J4: DF40C-20DS-0.4V_51, TinyTapeout:HRS_DF40C-20DP-0.4V_51, symbol TinyTapeout:DF40C-20DP-0.4V_51
- removed LAYOUT4: Standardized layout to allow for dual expansion b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, symbol psychogenic:LAYOUT
- removed MT3, MT4: MountingHole_Pad, MountingHole:MountingHole_3.2mm_M3_Pad, symbol Mechanical:MountingHole_Pad
- removed R26, R7: 1M, Resistor_SMD:R_0402_1005Metric, symbol psycomponents:PsyResistors_IEC/R_1M_0402_1005-14
- added D5: Yellow, LED_SMD:LED_0603_1608Metric, symbol Device:LED_Small
- added J14: Conn_02x16_Odd_Even, Connector_PinHeader_2.54mm:PinHeader_2x16_P2.54mm_Vertical, symbol Connector_Generic:Conn_02x16_Odd_Even
- added J16: Conn_02x05_Odd_Even, Connector_PinSocket_2.54mm:PinSocket_2x05_P2.54mm_Vertical, symbol Connector_Generic:Conn_02x05_Odd_Even
- added unit 5 of J5
- added unit 6 of J5
- added JP9: SolderJumper_2_Bridged, TinyTapeout:SolderJumper-2_0603, symbol Jumper:SolderJumper_2_Bridged
- added R32, R33, R34, R35, R36, R37, R38, R39, R40, R41, R42, R43: 10M, Resistor_SMD:R_0402_1005Metric, symbol psycomponents:PsyResistors_IEC/R_1M_0402_1005-14
- added R60: 510, Resistor_SMD:R_0402_1005Metric, symbol Device:R_Small
- added R61, R62, R63: 10k, Resistor_SMD:R_0402_1005Metric, symbol Device:R_Small
- C1: renamed from C7; JLC (none) -> C23829972; MPN CL10A105KA8NNNC -> GRM188D72A105KE01D
- C10: renamed from C8; value C_33p_0402_50V -> 33pF; JLC (none) -> C107005
- C11: renamed from C23; value 100nF -> 100n; JLC (none) -> C100072
- C12: renamed from C13; Characteristics 10u 10V XR 0603 -> 10u 0805; JLC (none) -> C408142
- C13: renamed from C14; JLC (none) -> C23829972; MPN CL10A105KA8NNNC -> GRM188D72A105KE01D
- C14: renamed from C15; Characteristics 10u 10V XR 0603 -> 10u 0805; JLC (none) -> C408142
- C15: renamed from C16; JLC (none) -> C23829972; MPN CL10A105KA8NNNC -> GRM188D72A105KE01D
- C16: renamed from C18; value 100nF -> 100n; JLC (none) -> C100072
- C17: renamed from C3; JLC (none) -> C576423; MPN (none) -> GCM188R72A682KA37D
- C18: renamed from C1; JLC (none) -> C23829972; MPN CL10A105KA8NNNC -> GRM188D72A105KE01D
- C19: renamed from C2; value 100nF -> 100n; JLC (none) -> C100072
- C2: renamed from C11; JLC (none) -> C23829972; MPN CL10A105KA8NNNC -> GRM188D72A105KE01D
- C20: renamed from C9; value 100nF -> 100n; JLC (none) -> C100072
- C21: renamed from C10; JLC (none) -> C23829972; MPN CL10A105KA8NNNC -> GRM188D72A105KE01D
- C22: renamed from C17; value 100nF -> 100n; JLC (none) -> C100072
- C23: renamed from C20; JLC (none) -> C23829972; MPN CL10A105KA8NNNC -> GRM188D72A105KE01D
- C24: value 100nF -> 100n; JLC (none) -> C100072
- C25: JLC (none) -> C23829972; MPN CL10A105KA8NNNC -> GRM188D72A105KE01D
- C3: renamed from C12; Characteristics 10u 10V XR 0805 -> 10u 0805; JLC (none) -> C408142
- C4: renamed from C19; Characteristics 22u 6V XR 0805 -> 22u 0805; JLC (none) -> C398931; MPN CL21A226KOQNNNG -> GRT21BR61E226ME13L
- C5: renamed from C21; value 100nF -> 100n; JLC (none) -> C100072
- C6: value C_33p_0402_50V -> 33pF; JLC (none) -> C107005
- C7: renamed from C4; value C_33p_0402_50V -> 33pF; JLC (none) -> C107005
- C8: renamed from C22; value 100nF -> 100n; JLC (none) -> C100072
- C9: renamed from C5; value C_33p_0402_50V -> 33pF; JLC (none) -> C107005
- D1, D2: footprint Resistor_SMD:R_0603_1608Metric -> Diode_SMD:D_0603_1608Metric; JLC (none) -> C6961594
- D3, D4: JLC (none) -> C6784997
- F1: JLC (none) -> C5468856
- FB1: JLC (none) -> C2649308
- J1: renamed from J5; JLC (none) -> C2927039
- J10: renamed from J15; Component Class (none) -> PMODSIL
- J11: renamed from J6; JLC (none) -> C5333437
- J12: renamed from J9; JLC (none) -> C5333437
- J13: renamed from J10; JLC (none) -> C5333437
- J2: renamed from J7; value 2x20_P2.54mm_Pinheader -> DF12NB(5.0)-50DP-0.5V(51); Characteristics (none) -> CONN HDR 50POS SMD GOLD; DNC do not change -> (none); JLC (none) -> C3020266; LCSC C3294478 -> (none); MPN 95157-440LF -> DF12NB(5.0)-50DP-0.5V(51); MPN_ALT PZ254-2-20-S -> (none)
- J3: renamed from J8; value 2x20_P2.54mm_Pinheader -> DF12NB(5.0)-60DP-0.5V(51); Characteristics (none) -> CONN HDR 60POS SMD GOLD; DNC do not change -> (none); JLC (none) -> C2847989; LCSC C3294478 -> (none); MPN 95157-440LF -> DF12NB(5.0)-60DP-0.5V(51); MPN_ALT PZ254-2-20-S -> (none)
- J4: renamed from J16; Component Class (none) -> PMODSIL
- J5: renamed from J1; value TT_HRS_BREAKOUT_REVA -> TT_HRS_BREAKOUT_REVB; footprint TinyTapeout:TT_HRS_CARRIER_REVA -> TinyTapeout:TT_HRS_CARRIER_REVC; symbol TinyTapeout:TT_HRS_BREAKOUT_REVA -> TinyTapeout:TT_HRS_BREAKOUT_REVB; now left out of the parts list
- J6: renamed from J13; Component Class (none) -> PMODSIL
- J8: renamed from J17; Component Class (none) -> PMODSIL
- J9: renamed from J14; Component Class (none) -> PMODSIL
- R1: renamed from R29; JLC (none) -> C25905
- R10: renamed from R1; JLC (none) -> C11702
- R12: renamed from R2; JLC (none) -> C25744
- R13: renamed from R3; JLC (none) -> C11702
- R14: renamed from R17; JLC (none) -> C25744
- R15: renamed from R27; JLC (none) -> C854484
- R16: renamed from R10; JLC (none) -> C25792; MPN (none) -> RC0402FR-0747KL
- R17: renamed from R41; JLC (none) -> C138040
- R18: renamed from R43; JLC (none) -> C276273
- R19: renamed from R18; JLC (none) -> C25744
- R2: renamed from R30; JLC (none) -> C25905
- R20: renamed from R32; JLC (none) -> C276273
- R21: renamed from R33; JLC (none) -> C276273
- R22: JLC (none) -> C11702
- R23: renamed from R34; JLC (none) -> C276273
- R24: renamed from R35; JLC (none) -> C276273
- R25: renamed from R36; JLC (none) -> C276273
- R26: renamed from R37; JLC (none) -> C276273
- R27: renamed from R38; JLC (none) -> C276273
- R28: renamed from R39; JLC (none) -> C276273
- R29: renamed from R31; JLC (none) -> C25905
- R3: renamed from R21; JLC (none) -> C11702
- R30: renamed from R40; JLC (none) -> C25744
- R31: renamed from R42; JLC (none) -> C25744
- R4: renamed from R16; JLC (none) -> C11702
- R44: renamed from R12; value 1M -> 10M; Characteristics RES SMD 1M OHM 1% 1/16W 0402 -> RES SMD 10M OHM 1% 1/16W 0402; JLC (none) -> C2076956; MPN AC0402FR-071ML -> CRCW040210M0FKEDC
- R45: renamed from R19; value 1M -> 10M; Characteristics RES SMD 1M OHM 1% 1/16W 0402 -> RES SMD 10M OHM 1% 1/16W 0402; JLC (none) -> C2076956; MPN AC0402FR-071ML -> CRCW040210M0FKEDC
- R46: renamed from R13; value 1M -> 10M; Characteristics RES SMD 1M OHM 1% 1/16W 0402 -> RES SMD 10M OHM 1% 1/16W 0402; JLC (none) -> C2076956; MPN AC0402FR-071ML -> CRCW040210M0FKEDC
- R47: renamed from R20; value 1M -> 10M; Characteristics RES SMD 1M OHM 1% 1/16W 0402 -> RES SMD 10M OHM 1% 1/16W 0402; JLC (none) -> C2076956; MPN AC0402FR-071ML -> CRCW040210M0FKEDC
- R48: renamed from R4; value 1M -> 10M; Characteristics RES SMD 1M OHM 1% 1/16W 0402 -> RES SMD 10M OHM 1% 1/16W 0402; JLC (none) -> C2076956; MPN AC0402FR-071ML -> CRCW040210M0FKEDC
- R49: renamed from R23; value 1M -> 10M; Characteristics RES SMD 1M OHM 1% 1/16W 0402 -> RES SMD 10M OHM 1% 1/16W 0402; JLC (none) -> C2076956; MPN AC0402FR-071ML -> CRCW040210M0FKEDC
- R5: renamed from R15; JLC (none) -> C11702
- R50: renamed from R5; value 1M -> 10M; Characteristics RES SMD 1M OHM 1% 1/16W 0402 -> RES SMD 10M OHM 1% 1/16W 0402; JLC (none) -> C2076956; MPN AC0402FR-071ML -> CRCW040210M0FKEDC
- R51: renamed from R24; value 1M -> 10M; Characteristics RES SMD 1M OHM 1% 1/16W 0402 -> RES SMD 10M OHM 1% 1/16W 0402; JLC (none) -> C2076956; MPN AC0402FR-071ML -> CRCW040210M0FKEDC
- R52: renamed from R6; value 1M -> 10M; Characteristics RES SMD 1M OHM 1% 1/16W 0402 -> RES SMD 10M OHM 1% 1/16W 0402; JLC (none) -> C2076956; MPN AC0402FR-071ML -> CRCW040210M0FKEDC
- R53: renamed from R25; value 1M -> 10M; Characteristics RES SMD 1M OHM 1% 1/16W 0402 -> RES SMD 10M OHM 1% 1/16W 0402; JLC (none) -> C2076956; MPN AC0402FR-071ML -> CRCW040210M0FKEDC
- R6: renamed from R14; JLC (none) -> C11702
- R7: renamed from R11; JLC (none) -> C11702
- R8: renamed from R9; JLC (none) -> C11702
- R9: renamed from R8; JLC (none) -> C11702
- SW1: renamed from SW4; JLC (none) -> C3293170
- SW2: renamed from SW1; JLC (none) -> C5525525
- SW3: renamed from SW2; JLC (none) -> C5525525
- SW4: renamed from SW3; JLC (none) -> C5525525
- U1: JLC (none) -> C15578
- U2: JLC (none) -> C22462656
- renumbered J2 to J7, R28 to R11
Connections:
- net +3V3: now also J5.L1 (3v3), J5.R10 (3v3), J5.R8 (3v3), J14.32 (Pin_32), J16.10 (Pin_10); no longer J5.L8 (3v3), J5.R5 (3v3)
- net ADC1: now also J16.3 (Pin_3)
- net ADC2: now also J16.4 (Pin_4)
- net ADC3: now also J16.5 (Pin_5)
- net ADC4: now also J16.8 (Pin_8)
- net ADC5: now also J16.7 (Pin_7)
- net GND: now also J5.L19 (GND), J5.L27 (GND), J5.L3 (GND), J5.L35 (GND), J5.L40 (GND), J5.L43 (GND), J5.L48 (GND), J5.L51 (GND), J5.L55 (GND), J5.L56 (GND), J5.L59 (GND), J5.L8 (GND), J5.R1 (GND), J5.R12 (GND), J5.R20 (GND), J5.R38 (GND), J5.R41 (GND), J5.R44 (GND), J5.R48 (GND), J8.7 (Pin_7), D5.1 (K), J14.1 (Pin_1), J14.14 (Pin_14), J14.17 (Pin_17), J14.22 (Pin_22), J14.25 (Pin_25), J14.30 (Pin_30), J14.31 (Pin_31), J14.6 (Pin_6), J14.9 (Pin_9), J16.1 (Pin_1), J16.2 (Pin_2), J16.6 (Pin_6), J16.9 (Pin_9), R32.1, R33.1, R34.1, R35.1, R36.2, R37.2, R38.2, R39.2, R40.2, R41.2, R42.2, R43.2, R61.2, R62.2, R63.2; no longer J5.L17 (GND), J5.L2 (GND), J5.L22 (GND), J5.L26 (GND), J5.L28 (GND), J5.L30 (GND), J5.L31 (GND), J5.L34 (GND), J5.L37 (GND), J5.L38 (GND), J5.L6 (GND), J5.R14 (GND), J5.R15 (GND), J5.R17 (GND), J5.R19 (GND), J5.R2 (GND), J5.R23 (GND), J5.R25 (GND), J5.R27 (GND), J5.R34 (GND), J5.R39 (GND), J5.R4 (GND), J5.R40 (GND), J5.R46 (GND), J5.R49 (GND), J5.R50 (GND), J5.R8 (GND), J8.5 (Pin_5), J8.9 (Pin_9)
- net VBUS: now also J5.R2 (VBUS), J5.R4 (VBUS); no longer J5.R1 (VBUS), J5.R3 (VBUS)
- net ctrl_ena: now also J5.R46 (ctrl_ena), J8.5 (Pin_5); no longer J5.L1 (ctrl_ena), J8.8 (Pin_8)
- net ctrl_sel_inc: now also J5.R47 (ctrl_inc), J8.4 (Pin_4); no longer J5.L4 (ctrl_inc), J8.7 (Pin_7)
- net project_clk: now also J5.L57 (proj_clk), JP9.2 (B); no longer J5.L36 (proj_clk), J9.3 (Pin_3)
- net res1: now also J5.R37 (RES1), J8.9 (Pin_9); no longer J5.L5 (RES1), J8.12 (Pin_12)
- net res2: now also J5.R35 (RES2), J8.10 (Pin_10); no longer J5.L7 (RES2), J8.11 (Pin_11)
- net res3: now also J5.R31 (RES3), J8.11 (Pin_11); no longer J5.L9 (RES3), J8.10 (Pin_10)
- net ui_in0: now also J5.L31 (ui_in[0]); no longer J5.L10 (ui_in[0])
- net ui_in1: now also J5.L33 (ui_in[1]); no longer J5.L12 (ui_in[1])
- net ui_in2: now also J5.L37 (ui_in[2]); no longer J5.L13 (ui_in[2])
- net ui_in3: now also J5.L39 (ui_in[3]); no longer J5.L14 (ui_in[3])
- net ui_in4: now also J5.L41 (ui_in[4]); no longer J5.L18 (ui_in[4])
- net ui_in5: now also J5.L45 (ui_in[5]); no longer J5.L20 (ui_in[5])
- net ui_in6: now also J5.L47 (ui_in[6]); no longer J5.L15 (ui_in[6])
- net ui_in7: now also J5.L49 (ui_in[7]); no longer J5.L33 (ui_in[7])
- net uio0: now also J5.L5 (uio[0]); no longer J5.L40 (uio[0])
- net uio1: now also J5.L7 (uio[1]); no longer J5.L39 (uio[1])
- net uio2: now also J5.L9 (uio[2]); no longer J5.R48 (uio[2])
- net uio3: now also J5.L13 (uio[3]); no longer J5.R47 (uio[3])
- net uio4: now also J5.L15 (uio[4]); no longer J5.R44 (uio[4])
- net uio5: now also J5.L17 (uio[5]); no longer J5.R43 (uio[5])
- net uio6: now also J5.L21 (uio[6]); no longer J5.R42 (uio[6])
- net uio7: now also J5.L23 (uio[7]); no longer J5.R41 (uio[7])
- net uo_out0: now also J5.R19 (uo_out[0]); no longer J5.R38 (uo_out[0])
- net uo_out1: now also J5.R17 (uo_out[1]); no longer J5.R37 (uo_out[1])
- net uo_out2: now also J5.R15 (uo_out[2]); no longer J5.R36 (uo_out[2])
- net uo_out3: now also J5.R13 (uo_out[3]); no longer J5.R35 (uo_out[3])
- net uo_out4: now also J5.R9 (uo_out[4]); no longer J5.R32 (uo_out[4])
- net uo_out5: now also J5.R7 (uo_out[5]); no longer J5.R31 (uo_out[5])
- net uo_out6: now also J5.R5 (uo_out[6]); no longer J5.R30 (uo_out[6])
- net uo_out7: now also J5.R3 (uo_out[7]); no longer J5.R29 (uo_out[7])
- net ~{ctrl_sel_rst}: now also J5.R43 (ctrl_~{rst}); no longer J5.L3 (ctrl_~{rst})
- net ~{project_rst}: now also J5.L53 (proj_~{rst}); no longer J5.L35 (proj_~{rst})
- net man_clk: now reaches C18.2, R14.2, R16.1, SW3.1
- net analog0 renamed N
- net N: now also J14.18 (Pin_18), J5.L34 (anN); no longer J5.L19 (an0)
- net analog1 renamed P
- net P: now also J14.19 (Pin_19), J5.L36 (anP); no longer J5.L21 (an1)
- net analog10 renamed X
- net X: now also J14.29 (Pin_29), J5.L58 (anX); no longer J5.R18 (an10)
- removed net analog11: J5.R16 (an11)
- net analog2 renamed Q
- net Q: now also J14.20 (Pin_20), J5.L38 (anQ); no longer J5.L23 (an2)
- net analog3 renamed R
- net R: now also J14.21 (Pin_21), J5.L42 (anR); no longer J5.L25 (an3)
- net analog4 renamed S
- net S: now also J14.24 (Pin_24), J5.L44 (anS); no longer J5.L27 (an4)
- removed net analog5: J5.L29 (an5)
- net analog6 renamed T
- net T: now also J14.23 (Pin_23), J5.L46 (anT); no longer J5.R26 (an6)
- net analog7 renamed U
- net U: now also J14.26 (Pin_26), J5.L50 (anU); no longer J5.R24 (an7)
- net analog8 renamed V
- net V: now also J14.27 (Pin_27), J5.L52 (anV); no longer J5.R22 (an8)
- net analog9 renamed W
- net W: now also J14.28 (Pin_28), J5.L54 (anW); no longer J5.R20 (an9)
- new net: D5.2 (A), R60.2
- new net: J9.3 (Pin_3), JP9.1 (A)
- new net A: J14.2 (Pin_2), J5.L2 (anA), R32.2
- new net B: J14.3 (Pin_3), J5.L4 (anB), R34.2
- new net C: J14.4 (Pin_4), J5.L6 (anC), R36.1
- new net D: J14.5 (Pin_5), J5.L10 (anD), R38.1
- new net E: J14.8 (Pin_8), J5.L12 (anE), R40.1
- new net F: J14.7 (Pin_7), J5.L14 (anF), R42.1
- new net G: J14.10 (Pin_10), J5.L18 (anG), R33.2
- new net H: J14.11 (Pin_11), J5.L20 (anH), R35.2
- new net J: J14.12 (Pin_12), J5.L22 (anJ), R37.1
- new net K: J14.13 (Pin_13), J5.L26 (anK), R39.1
- new net L: J14.16 (Pin_16), J5.L28 (anL), R41.1
- new net M: J14.15 (Pin_15), J5.L30 (anM), R43.1
- new net RPLED: R60.1
- new net mng0: J5.R42 (mng00)
- new net mng1: J5.R40 (mng01)
- new net mng2: J5.R36 (mng02)
- new net mng3: J5.R30 (mng03)
- new net mng4: J5.R26 (mng04), R61.1
- new net mng5: J5.R22 (mng05), R62.1
- new net mng6: J5.R18 (mng06)
- new net mng7: J5.R16 (mng07), R63.1
- new net res0: J5.R39 (RES0), J8.8 (Pin_8)
- new net res4: J5.R29 (RES4), J8.12 (Pin_12)
- no-connect marks 3 -> 8
Other:
- sheet RP2350 ports: added GPIO40; removed ADC0
- note added: ""Management" pins go to breakout board, function dependant on specific carrier inserted."
- note added: "DB analog header"
- note added: "Edge connectors: Management"
- note added: "Edge connectors: Project"
- note added: "Project MUX, power and reserved pins available on this header"
- note added: "Tiny Tapeout Demoboard v3"
- note added: "ck"
- note added: "from PMOD J11"
- note added: "from PMOD J12"
- note added: "from PMOD J13"
- note added: "rx"
- note added: "tx"
- note added: "~{cs}"
- note removed: "Analog Bank A"
- note removed: "Analog Bank B"
- note removed: "Board edge connectors (pinheaders)"
- note removed: "Expansion headers placed on each side, in line with analog, 10mm to right when facing breakout."
- note removed: "Tiny Tapeout Demoboard v3 (PRELIMINARY)"
- note removed: "from PMOD J3"
- note removed: "from PMOD J5"
- note removed: "from PMOD J6"
- title: Tiny Tapeout Demoboard v3 (PRELIMINARY) -> Tiny Tapeout Demoboard v3
- moved on the sheet: C1, C10, C11, C12, C13, C14, C15, C16, C17, C19, C2, C3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
